File: hardware/keyboard-classic/kbd-classic.kicad_pcb (KiCad board)
At the start: 2 copper layers, 307.3 x 107.7 mm, 137 parts, among them J1 Controller, SW1 Clear, SW10 Bracket_Open, SW11 6, SW12 Y, SW13 Return, SW14 Dash, SW15 5, SW16 T, SW17 Line Feed, SW18 Colon, SW19 4, SW2 Repeat, SW20 R, SW21 O, SW22 0, SW23 3, SW24 E, SW25 L, SW26 9, SW27 2, SW28 W, SW29 Period, SW3 Tilde, SW30 8, SW31 1, SW32 @ (OSI shift lock), SW33 Break, SW34 Rubout (OSI Break), SW35 R_Shift, SW36 P, SW37 Comma, SW38 K, SW39 L_Shift, SW4 I, SW40 Semicolon, SW41 M, SW42 J, SW43 Fwd_Slash, SW44 N, SW45 H, SW46 SPACE, SW47 B, SW48 G, SW49 ESC, SW5 Here_is, SW50 Z, SW51 V, SW52 F, SW53 CTRL, SW54 A, SW55 C, SW56 D, SW57 Backslash, SW58 Q, SW59 X, SW6 Bracket_Close, SW60 S, SW61 Power light, SW7 7, SW8 U, SW9 Caps_Lock

Commit message: OSI mounting holes
- Add OSI-compatible mounting holes.
- Adjust keyboard and aligner holes to make room for the OSI mounting holes
- Change "Universal Keyboard" to "Unified Keyboard" in the design files.
Parts:
- removed the REF** at (363.2, 171.4)
- removed the REF** at (107.8, 171.4)
- removed the REF** at (284.6, 171.4)
- added REF**: MountingHole_3.5mm, MountingHole:MountingHole_3.5mm, F.Cu at (306.8, 73.1)
- added REF**: MountingHole_3.5mm, MountingHole:MountingHole_3.5mm, F.Cu at (102.7, 171.4)
- added REF**: MountingHole_3.5mm, MountingHole:MountingHole_3.5mm, F.Cu at (289.7, 171.4)
- added REF**: MountingHole_3.5mm, MountingHole:MountingHole_3.5mm, F.Cu at (358.1, 171.4)
- added REF**: MountingHole_3.5mm, MountingHole:MountingHole_3.5mm, F.Cu at (87.1, 73.1)
- added REF**: MountingHole_3.5mm, MountingHole:MountingHole_3.5mm, F.Cu at (196.9, 73.1)
- added REF**: MountingHole_3.5mm, MountingHole:MountingHole_3.5mm, F.Cu at (111.0, 166.5)
- added REF**: MountingHole_3.5mm, MountingHole:MountingHole_3.5mm, F.Cu at (282.9, 166.5)
Routing:
- net Net-(J1-Pad4): track 231.7 -> 238.5 mm
- net Net-(J1-Pad6): track 233.7 -> 240.2 mm
- net Net-(J1-Pad2): track 227.2 -> 233.7 mm
- net Net-(J1-Pad8): track 240.5 -> 246.6 mm
- net /Col6: track 404.8 -> 408.9 mm
- net /Col5: track 449.1 -> 453.0 mm
- net /Col4: track 306.3 -> 305.0 mm
Other:
- board size 307.3 x 107.7 mm -> 307.3 x 112.8 mm
- board text added: "Unified Keyboard Rev 1.2 http://osiweb.org"
- board text removed: "Universal Keyboard Rev 1.2 http://osiweb.org"

Commit message: Swap "O" (Cap O) and "0" (zero) keys
The "0" and "O" keys were swapped on the PCB, requiring a keymap fix for the
ASCII adapter.  The swapped keys would not be an issue for a keyscanning ASCII
converter, but would preclude use in OSI systems, so this fix puts the keys
back in position compatible with OSI.
Parts:
- moved SW21 21.4 mm to (249.3, 108.8)
- moved SW22 21.4 mm to (259.1, 89.8)
- moved D22 21.4 mm to (258.8, 105.0)
- moved D23 21.4 mm to (268.6, 86.0)
Routing:
- net /Row6: track 274.7 -> 255.5 mm
- net /Row5: track 277.6 -> 275.8 mm, vias 3 -> 2
- net /Row4: track 405.4 -> 406.8 mm
Other:
- board text added: "Unified Keyboard Rev 1.3 http://osiweb.org"
- board text removed: "Unified Keyboard Rev 1.2 http://osiweb.org"

Commit message: Finalize layout and mounting
- Add apple 2 mounting slots (and stretch PCB to accommodate slots
- Add pass-through holes in aligners for OSI keyboard spacers
- Move 'ESC' key next to '1' key
- Add TAB key next to Q key
- remove 'here is' and finalize "helper" keys along left side of keyboard
- move legends off of PCB traces
- update to release 1.3
Parts:
- removed the REF** at (306.8, 73.1)
- removed the REF** at (130.3, 174.3)
- removed the REF** at (130.3, 159.0)
- removed the REF** at (87.1, 73.1)
- removed the REF** at (196.9, 73.1)
- removed the REF** at (111.0, 166.5)
- removed the REF** at (282.9, 166.5)
- removed the REF** at (165.2, 176.2)
- removed the REF** at (228.7, 176.2)
- added D1: 1N4148, Diode_THT:D_DO-35_SOD27_P7.62mm_Horizontal, F.Cu at (78.1, 86.0)
- added OSI: MountingHole_3.5mm, MountingHole:MountingHole_3.5mm, F.Cu at (306.8, 73.1)
- added OSI: MountingHole_3.5mm, MountingHole:MountingHole_3.5mm, F.Cu at (87.1, 73.1)
- added OSI: MountingHole_3.5mm, MountingHole:MountingHole_3.5mm, F.Cu at (196.9, 73.1)
- added OSI: MountingHole_3.5mm, MountingHole:MountingHole_3.5mm, F.Cu at (111.0, 166.5)
- added OSI: MountingHole_3.5mm, MountingHole:MountingHole_3.5mm, F.Cu at (282.9, 166.5)
- added OSI: MountingHole_3.5mm, MountingHole:MountingHole_3.5mm, F.Cu at (165.2, 176.2)
- added OSI: MountingHole_3.5mm, MountingHole:MountingHole_3.5mm, F.Cu at (228.7, 176.2)
- added SW62: ESC, unikbd:Key_MX, F.Cu at (68.6, 89.8)
- added Stabilizer: MountingHole_3.5mm, MountingHole:MountingHole_3.5mm, F.Cu at (130.3, 174.3)
- added Stabilizer: MountingHole_3.5mm, MountingHole:MountingHole_3.5mm, F.Cu at (130.3, 159.0)
- SW1: value Clear -> RT Arrow
- SW2: value Repeat -> LT Arrow
- SW49: value ESC -> TAB
- SW5: value Here_is -> Repeat
Routing:
- net /Col4: track 305.0 -> 387.7 mm
- net /Row0: track 353.3 -> 376.8 mm
- net /Col1: track 373.1 -> 361.5 mm
- net Net-(D1-Pad2): track 0.00 -> 9.72 mm
- net /Col7: track 382.7 -> 390.0 mm
- net /Row1: track 349.1 -> 355.4 mm
- net /Row6: track 255.5 -> 259.4 mm
- net Net-(J1-Pad16): track 64.8 -> 68.5 mm
- net Net-(J1-Pad20): track 53.3 -> 56.4 mm
- net /Col6: track 408.9 -> 411.9 mm
- net /Col0: track 129.8 -> 132.3 mm
- net /Row4: track 406.8 -> 405.4 mm
- net /Row7: track 313.7 -> 312.7 mm
- net Net-(J1-Pad10): track 63.2 -> 62.3 mm
- net Net-(J1-Pad14): track 60.6 -> 61.5 mm
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Other:
- board size 307.3 x 112.8 mm -> 365.4 x 112.8 mm

Commit message: Trace fixes
- removed extraneous unconnected traces
- straightened an off-angle trace that was violating clearance.
Routing:
- net /Row2: track 374.8 -> 319.7 mm
- net /Row3: track 323.0 -> 290.4 mm
- net /Row4: track 405.4 -> 392.2 mm
- net /Col3: track 302.8 -> 299.4 mm

Commit message: Keyboard layout updates
- Add extra key to the left side of row 4 to permit "inverted T" for those who
  want it.

- Tiny shifts of several keys to correct key distances

- Include mounting holes with daughter board connector, to ensure consistency.
Parts:
- removed OSI (x7): MountingHole_3.5mm, MountingHole:MountingHole_3.5mm
- removed the Stabilizer at (130.3, 174.3)
- removed the Stabilizer at (130.3, 159.0)
- added D33: LED, LED_THT:LED_D5.0mm, F.Cu at (368.6, 127.9)
- added D35: 1N4148, Diode_THT:D_DO-35_SOD27_P7.62mm_Horizontal, F.Cu at (378.0, 143.1)
- added REF**: OSI mounting holes, unikbd:OSI mounting holes, F.Cu at (197.2, 166.0)
- added SW63: Spare, unikbd:Key_MX, F.Cu at (368.6, 146.9)
- added Stabilizer: MountingHole_3.5mm, MountingHole:MountingHole_3.5mm, F.Cu at (130.5, 174.3)
- added Stabilizer: MountingHole_3.5mm, MountingHole:MountingHole_3.5mm, F.Cu at (130.5, 159.0)
- moved D2 1.89 mm to (358.9, 143.1)
- moved SW12 0.28 mm to (192.4, 108.8)
- moved SW17 0.28 mm to (287.6, 108.8)
- moved SW20 0.28 mm to (154.3, 108.8)
- moved SW21 0.28 mm to (249.5, 108.8)
- moved SW36 0.28 mm to (268.6, 108.8)
- moved SW8 0.28 mm to (211.4, 108.8)
- moved SW28 0.28 mm to (116.2, 108.8)
- moved SW58 0.28 mm to (97.1, 108.8)
- moved SW16 0.28 mm to (173.3, 108.8)
- moved SW24 0.28 mm to (135.2, 108.8)
- moved SW4 0.28 mm to (230.5, 108.8)
- moved SW13 0.24 mm to (311.5, 108.8)
- moved REF** 0.22 mm to (263.8, 174.3)
- moved REF** 0.22 mm to (263.8, 159.0)
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Routing:
- net /Row3: track 290.4 -> 341.9 mm, vias 1 -> 2
- net Net-(D33-Pad2): track 114.6 -> 150.8 mm
- net Net-(D33-Pad1): track 113.1 -> 146.7 mm
- net /Col0: track 132.3 -> 153.9 mm
- net Net-(D35-Pad2): track 0.00 -> 9.47 mm
- net /Col7: track 390.0 -> 385.5 mm
- net Net-(D2-Pad2): track 11.3 -> 9.49 mm
- net /Row2: track 319.7 -> 321.5 mm
- net Net-(J1-Pad12): track 60.7 -> 60.8 mm, vias 0 -> 1
Other:
- board text added: "Distances: Vertical: 0.75 inch Horizontal (1x - 1x): 0.75 inch Horizontal (1x - 1.5x): 0.9375 inch Horizontal (Row 1 left key -> Row 2 left key): 0.375 inch Horizontal (Row 2 left key -> Row 3 left key): 0.1875 inch Horizontal (Row 3 left key -> Row 4 left key): 0.1875 inch Horizontal (Row 4 left key -> Row 5 left key): -0.1875 inch Horizontal (Row 5 left key -> Space bar): 4.5 inch"
- board text removed: "Distances: Vertical: 0.75 inch Horizontal (1x - 1x): 0.75 inch Horizontal (1x - 1.5x): 0.939 inch Horizontal (Row 1 left key -> Row 2 left key): -0.379 inch Horizontal (Row 2 left key -> Row 3 left key): 0.187 inch Horizontal (Row 3 left key -> Row 4 left key): 0.186 inch Horizontal (Row 4 left key -> space bar): 4.310 inch"

Commit message: Fix wrong apple-II mount dimensions
- pulled in the right border and mounting holes for Apple-II mounting dimensions
- modified the "~^" key courtyard to allow closer positioning of the upper right
  Apple II Mounting hole.  (The ~^ key is not installed in an Apple II keyboard)
- Moved tracks and diodes as needed to keep everything in the new outline.
Parts:
- moved D4 11.1 mm to (370.6, 95.0)
- moved D35 8.84 mm to (372.8, 135.9), turned to 180 degrees
Routing:
- net Net-(D33-Pad1): track 146.7 -> 125.7 mm
- net Net-(D33-Pad2): track 150.8 -> 129.9 mm
- net /Row6: track 259.4 -> 276.0 mm
- net Net-(D4-Pad2): track 9.56 -> 22.5 mm
- net Net-(D35-Pad2): track 9.47 -> 20.6 mm
- net /Row3: track 341.9 -> 339.0 mm
Other:
- board size 365.4 x 112.8 mm -> 348 x 112.8 mm
