File: hardware/keyboard-classic/kbd-classic.kicad_pcb (KiCad board)
At the start: 2 copper layers, 346.1 x 116.8 mm, 144 parts, among them J1 Controller, SW1 RT Arrow, SW10 Bracket_Open, SW11 6, SW12 Y, SW13 Return, SW14 Dash, SW15 5, SW16 T, SW17 Line_Feed, SW18 Colon, SW19 4, SW2 LT Arrow, SW20 R, SW21 O, SW22 0, SW23 3, SW24 E, SW25 L, SW26 9, SW27 2, SW28 W, SW29 Period, SW3 Tilde, SW30 8, SW31 1, SW32 @ (OSI ShiftLock), SW33 Break, SW34 Rubout (OSI Break), SW35 R_Shift, SW36 P, SW37 Comma, SW38 K, SW39 L_Shift, SW4 I, SW40 Semicolon, SW41 M, SW42 J, SW43 Fwd_Slash, SW44 N, SW45 H, SW46 SPACE, SW47 B, SW48 G, SW49 TAB, SW5 Repeat, SW50 Z, SW51 V, SW52 F, SW53 CTRL, SW54 A, SW55 C, SW56 D, SW57 Backslash, SW58 Q, SW59 X, SW6 Bracket_Close, SW60 S, SW61 Power Light, SW62 ESC, SW63 Spare, SW7 7, SW8 U, SW9 Caps_Lock

Commit message: mechanical fit and buildability fixes
- Moved header slightly forward

- Moved interface mount holes do reduce interference with case mount holes

- For all keys in classic keyboard, add option for either through-hole or SMT
diodes and resistors.
Parts:
- removed the REF** at (289.7, 171.4)
- removed the REF** at (358.1, 171.4)
- removed the REF** at (349.0, 77.5)
- removed the REF** at (300.7, 77.5)
- added R4: 470, Resistor_SMD:R_0805_2012Metric, B.Cu at (67.1, 157.2)
- added R5: 470, Resistor_SMD:R_0805_2012Metric, B.Cu at (318.1, 171.9)
- added R6: 470, Resistor_SMD:R_0805_2012Metric, B.Cu at (368.0, 112.0)
- D1, D10, D11, D12, D13, D14, D15, D16, D17, D18, D19, D2, D20, D21, D22, D23, D24, D25, D26, D27, D28, D29, D3, D30, D31, D32, D34, D35, D36, D37, D38, D39, D4, D40, D41, D42, D43, D44, D45, D46, D47, D48, D49, D5, D50, D51, D52, D53, D54, D55, D56, D57, D58, D59, D6, D60, D61, D7, D8, D9: footprint Diode_THT:D_DO-35_SOD27_P7.62mm_Horizontal -> unikbd:diode-combined
- J1: footprint Connector_PinHeader_2.54mm:PinHeader_2x20_P2.54mm_Vertical -> unikbd:kbd_header_and_mounting_holes; moved to F.Cu
- moved R2 5.72 mm to (313.0, 171.8)
- moved J1 2.56 mm to (301.0, 163.9), turned to 90 degrees
- moved D4 2.02 mm to (366.2, 94.2)
- moved D35 1.32 mm to (373.9, 136.8)
Routing:
- net /Col3: track 298.6 -> 346.6 mm, vias 2 -> 4
- net /Col2: track 471.7 -> 500.6 mm, vias 4 -> 8
- net /Col4: track 387.7 -> 414.4 mm, vias 3 -> 2
- net /Col6: track 412.3 -> 426.4 mm, vias 4 -> 6
- net /Row0: track 377.1 -> 363.0 mm
- net Net-(D63-Pad2): track 110.9 -> 100.1 mm
- net Net-(J1-Pad20): track 56.4 -> 46.0 mm, vias 0 -> 2
- net Net-(D33-Pad2): track 188.2 -> 180.4 mm, vias 2 -> 1
- net Net-(D33-Pad1): track 171.2 -> 165.1 mm
- net /Col5: track 453.0 -> 447.3 mm, vias 5 -> 6
- net /Row3: track 348.6 -> 343.2 mm
- net Net-(J1-Pad14): track 10.7 -> 15.1 mm
- net Net-(J1-Pad6): track 259.7 -> 264.1 mm
- net Net-(J1-Pad12): track 61.9 -> 57.9 mm
- net Net-(J1-Pad10): track 63.6 -> 59.7 mm
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Other:
- board text added: "Unified Keyboard Rev 1.8 http://osiweb.org"
- board text removed: "Unified Keyboard Rev 1.7 http://osiweb.org"

Commit message: Add/update keyboard cutout outlines for Full ASCII, OSI, and Apple
Other:
- board text added: "Apple II keyboard cutout"
- board text added: "Full ASCII keyboard cutout"
- board text added: "Keyboard Cutout layers: Full ASCII: Eco1.User Apple II+: Dwgs.User OSI: Eco2.User"
- board text added: "OSI 542 keyboard cutout"
Changed lines of the file:
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@@
   (general
     (thickness 1.6)
-    (drawings 44)
+    (drawings 81)
     (tracks 1209)
     (zones 0)
@@
   (layers
     (0 F.Cu signal)
-    (31 B.Cu signal)
-    (32 B.Adhes user)
-    (33 F.Adhes user)
-    (34 B.Paste user)
-    (35 F.Paste user)
-    (36 B.SilkS user)
+    (31 B.Cu signal hide)
+    (32 B.Adhes user hide)
+    (33 F.Adhes user hide)
+    (34 B.Paste user hide)
+    (35 F.Paste user hide)
+    (36 B.SilkS user hide)
     (37 F.SilkS user)
-    (38 B.Mask user)
-    (39 F.Mask user)
+    (38 B.Mask user hide)
+    (39 F.Mask user hide)
     (40 Dwgs.User user)
     (41 Cmts.User user)
@@
     (43 Eco2.User user)
     (44 Edge.Cuts user)
-    (45 Margin user)
-    (46 B.CrtYd user)
-    (47 F.CrtYd user)
-    (48 B.Fab user)
-    (49 F.Fab user)
+    (45 Margin user hide)
+    (46 B.CrtYd user hide)
+    (47 F.CrtYd user hide)
+    (48 B.Fab user hide)
+    (49 F.Fab user hide)
   )
   (setup
@@
     (pad 1 np_thru_hole circle (at 0 0) (size 3.5 3.5) (drill 3.5) (layers *.Cu *.Mask))
   )
+  (gr_text "Full ASCII keyboard cutout" (at 120.396 184.6326) (layer Eco1.User)
+    (effects (font (size 2.54 2.54) (thickness 0.3048)) (justify left))
+  )
+  (gr_text "OSI 542 keyboard cutout" (at 234.315 184.6326) (layer Eco2.User)
+    (effects (font (size 2.54 2.54) (thickness 0.3048)) (justify left))
+  )
+  (gr_text "Apple II keyboard cutout" (at 179.351214 184.6326) (layer Dwgs.User)
+    (effects (font (size 2.54 2.54) (thickness 0.3048)) (justify left))
+  )
+  (gr_line (start 339.65388 137.80516) (end 320.60388 137.80516) (layer Eco2.User) (width 0.15))
+  (gr_line (start 339.65388 118.75516) (end 339.65388 137.80516) (layer Eco2.User) (width 0.15))
+  (gr_line (start 320.60388 137.80516) (end 320.60388 156.09316) (layer Eco2.User) (width 0.15))
+  (gr_text "Keyboard Cutout layers:\nFull ASCII: Eco1.User\nApple II+: Dwgs.User\nOSI: Eco2.User" (at 38.4175 200.57618) (layer Cmts.User)
+    (effects (font (size 2.54 2.54) (thickness 0.3048)) (justify left))
+  )
+  (gr_line (start 325.36638 118.75516) (end 339.65388 118.75516) (layer Eco2.User) (width 0.15))
+  (gr_line (start 325.36638 80.65516) (end 325.36638 118.75516) (layer Eco2.User) (width 0.15))
+  (gr_line (start 320.60388 118.75516) (end 320.60388 156.09316) (layer Dwgs.User) (width 0.15))
+  (gr_line (start 325.36638 118.75516) (end 320.60388 118.75516) (layer Dwgs.User) (width 0.15))
+  (gr_line (start 325.36638 80.65516) (end 325.36638 118.75516) (layer Dwgs.User) (width 0.15))
+  (gr_line (start 77.71638 98.94316) (end 77.71638 80.65516) (layer Dwgs.User) (width 0.15))
+  (gr_line (start 92.00388 156.09316) (end 92.00388 175.14316) (layer Dwgs.User) (width 0.15))
+  (gr_line (start 73.71588 175.14316) (end 92.00388 175.14316) (layer Dwgs.User) (width 0.15))
+  (gr_line (start 77.71638 98.94316) (end 68.95338 98.94316) (layer Dwgs.User) (width 0.15))
+  (gr_line (start 59.42838 80.65516) (end 325.36638 80.65516) (layer Dwgs.User) (width 0.15))
+  (gr_line (start 320.60388 156.09316) (end 272.97888 156.09316) (layer Dwgs.User) (width 0.15))
+  (gr_line (start 272.97888 156.09316) (end 272.97888 175.14316) (layer Dwgs.User) (width 0.15))
+  (gr_line (start 272.923 175.14316) (end 121.34088 175.14316) (layer Dwgs.User) (width 0.15))
+  (gr_line (start 121.34088 175.133) (end 121.34088 156.09316) (layer Dwgs.User) (width 0.15))
+  (gr_line (start 121.34088 156.09316) (end 92.00388 156.09316) (layer Dwgs.User) (width 0.15))
+  (gr_line (start 73.71588 117.99316) (end 68.95338 117.99316) (layer Dwgs.User) (width 0.15))
+  (gr_line (start 68.95338 117.99316) (end 68.95338 98.94316) (layer Dwgs.User) (width 0.15))
+  (gr_line (start 73.71588 175.14316) (end 73.71588 117.99316) (layer Dwgs.User) (width 0.15))
+  (gr_line (start 73.71588 156.09316) (end 73.71588 117.99316) (layer Eco2.User) (width 0.15))
+  (gr_line (start 272.923 175.14316) (end 121.34088 175.14316) (layer Eco2.User) (width 0.15))
+  (gr_line (start 59.42838 98.94316) (end 68.95338 98.94316) (layer Eco2.User) (width 0.15))
+  (gr_line (start 59.42838 80.65516) (end 325.36638 80.65516) (layer Eco2.User) (width 0.15))
+  (gr_line (start 272.97888 156.09316) (end 272.97888 175.14316) (layer Eco2.User) (width 0.15))
+  (gr_line (start 59.42838 98.94316) (end 59.42838 80.65516) (layer Eco2.User) (width 0.15))
+  (gr_line (start 68.95338 117.99316) (end 68.95338 98.94316) (layer Eco2.User) (width 0.15))
+  (gr_line (start 73.71588 117.99316) (end 68.95338 117.99316) (layer Eco2.User) (width 0.15))
+  (gr_line (start 121.34088 156.09316) (end 73.71588 156.09316) (layer Eco2.User) (width 0.15))
+  (gr_line (start 121.34088 175.133) (end 121.34088 156.09316) (layer Eco2.User) (width 0.15))
+  (gr_line (start 320.60388 156.09316) (end 272.97888 156.09316) (layer Eco2.User) (width 0.15))
+  (gr_line (start 358.70388 137.80516) (end 358.70388 156.09316) (layer Eco1.User) (width 0.15))
   (gr_line (start 379.73 132.715) (end 379.73 180.34) (layer Edge.Cuts) (width 0.1016))
   (gr_line (start 370.21738 94.615) (end 379.73 94.615) (layer Edge.Cuts) (width 0.1016))
   (gr_line (start 370.21738 132.715) (end 379.73 132.715) (layer Edge.Cuts) (width 0.1016))
   (gr_line (start 370.21738 94.615) (end 370.21738 132.715) (layer Edge.Cuts) (width 0.1016))
-  (gr_line (start 377.75388 137.80516) (end 358.70388 137.80516) (layer B.Fab) (width 0.15))
-  (gr_line (start 377.75388 137.80516) (end 377.75388 156.09316) (layer B.Fab) (width 0.15))
+  (gr_line (start 377.75388 137.80516) (end 358.70388 137.80516) (layer Eco1.User) (width 0.15))
+  (gr_line (start 377.75388 137.80516) (end 377.75388 156.09316) (layer Eco1.User) (width 0.15))
   (gr_arc (start 376.64738 89.79916) (end 376.64738 91.57716) (angle -180) (layer Edge.Cuts) (width 0.1016))
   (gr_arc (start 376.64738 165.99916) (end 376.64738 167.77716) (angle -180) (layer Edge.Cuts) (width 0.1016))
-  (gr_line (start 73.71588 175.14316) (end 73.71588 117.99316) (layer B.Fab) (width 0.15))
-  (gr_line (start 59.42838 98.94316) (end 68.95338 98.94316) (layer B.Fab) (width 0.15))
+  (gr_line (start 73.71588 175.14316) (end 73.71588 117.99316) (layer Eco1.User) (width 0.15))
+  (gr_line (start 59.42838 98.94316) (end 68.95338 98.94316) (layer Eco1.User) (width 0.15))
   (gr_line (start 43.17238 88.02116) (end 33.64738 88.02116) (layer Edge.Cuts) (width 0.1016))
   (gr_line (start 43.17238 164.22116) (end 33.64738 164.22116) (layer Edge.Cuts) (width 0.1016))
@@
     (effects (font (size 1.524 1.524) (thickness 0.1778)))
   )
-  (gr_line (start 358.70388 117.99316) (end 363.46638 117.99316) (layer B.Fab) (width 0.15))
-  (gr_line (start 73.71588 175.14316) (end 92.00388 175.14316) (layer B.Fab) (width 0.15))
-  (gr_line (start 92.00388 156.09316) (end 92.00388 175.14316) (layer B.Fab) (width 0.15))
-  (gr_line (start 358.70388 117.99316) (end 358.70388 137.80516) (layer B.Fab) (width 0.15))
-  (gr_line (start 363.46638 80.65516) (end 363.46638 117.99316) (layer B.Fab) (width 0.15))
-  (gr_line (start 59.42838 98.94316) (end 59.42838 80.65516) (layer B.Fab) (width 0.15))
-  (gr_line (start 68.95338 117.99316) (end 68.95338 98.94316) (layer B.Fab) (width 0.15))
-  (gr_line (start 73.71588 117.99316) (end 68.95338 117.99316) (layer B.Fab) (width 0.15))
-  (gr_line (start 121.34088 156.09316) (end 92.00388 156.09316) (layer B.Fab) (width 0.15))
-  (gr_line (start 121.34088 175.133) (end 121.34088 156.09316) (layer B.Fab) (width 0.15))
-  (gr_line (start 272.923 175.14316) (end 121.34088 175.14316) (layer B.Fab) (width 0.15))
-  (gr_line (start 272.97888 156.09316) (end 272.97888 175.14316) (layer B.Fab) (width 0.15))
-  (gr_line (start 377.75388 156.09316) (end 272.97888 156.09316) (layer B.Fab) (width 0.15))
-  (gr_line (start 59.42838 80.65516) (end 363.46638 80.65516) (layer B.Fab) (width 0.15))
+  (gr_line (start 358.70388 117.99316) (end 363.46638 117.99316) (layer Eco1.User) (width 0.15))
+  (gr_line (start 73.71588 175.14316) (end 92.00388 175.14316) (layer Eco1.User) (width 0.15))
+  (gr_line (start 92.00388 156.09316) (end 92.00388 175.14316) (layer Eco1.User) (width 0.15))
+  (gr_line (start 358.70388 117.99316) (end 358.70388 137.80516) (layer Eco1.User) (width 0.15))
+  (gr_line (start 363.46638 80.65516) (end 363.46638 117.99316) (layer Eco1.User) (width 0.15))
+  (gr_line (start 59.42838 98.94316) (end 59.42838 80.65516) (layer Eco1.User) (width 0.15))
+  (gr_line (start 68.95338 117.99316) (end 68.95338 98.94316) (layer Eco1.User) (width 0.15))
+  (gr_line (start 73.71588 117.99316) (end 68.95338 117.99316) (layer Eco1.User) (width 0.15))
+  (gr_line (start 121.34088 156.09316) (end 92.00388 156.09316) (layer Eco1.User) (width 0.15))
+  (gr_line (start 121.34088 175.133) (end 121.34088 156.09316) (layer Eco1.User) (width 0.15))
+  (gr_line (start 272.923 175.14316) (end 121.34088 175.14316) (layer Eco1.User) (width 0.15))
+  (gr_line (start 272.97888 156.09316) (end 272.97888 175.14316) (layer Eco1.User) (width 0.15))
+  (gr_line (start 377.75388 156.09316) (end 272.97888 156.09316) (layer Eco1.User) (width 0.15))
+  (gr_line (start 59.42838 80.65516) (end 363.46638 80.65516) (layer Eco1.User) (width 0.15))
   (gr_line (start 33.64738 180.34) (end 379.73 180.34) (layer Edge.Cuts) (width 0.1))
   (gr_line (start 379.73 63.5) (end 33.64738 63.5) (layer Edge.Cuts) (width 0.1))

Commit message: Multiple fixes for keyboard PCB
- in combined CherryMX/futaba footprints, moved cherry pads down 1 mil and
futaba pads up 2 mil, to reduce risk of shortin of LED pads with futaba pad.
Adjusted all aligners accordingly

- Fixed centroid for combined diode footprint and adjusted PCB placement on
classic and SOL keyboards accordingly.

- Moved SMT pads in combined diode footprint to top layer, so pick & place file
will be usable.

- changes to futaba stabilizer design.  Longer post adapter passes through slots
in keyboard and aligner.

- Changed futaba post thickness gauge from board outline to a slot to improve
tolerance.

- Moved spacebar stabilizer bending guide to edge of PCB, in order to make it
more useful in bending PCBs.

- Changed Apple II mounting slots on classic keyboard from horizontal to
vertical orientation, to accommodate the different spacing offets due to the use
of spacers in angled mounting threads.
Parts:
- D1, D10, D11, D12, D13, D14, D15, D16, D17, D18, D19, D2, D20, D21, D22, D23, D24, D25, D26, D27, D28, D29, D3, D30, D31, D32, D34, D35, D36, D37, D38, D39, D4, D40, D41, D42, D43, D44, D45, D46, D47, D48, D49, D5, D50, D51, D52, D53, D54, D55, D56, D57, D58, D59, D6, D60, D61, D7, D8, D9: moved to B.Cu
- moved D4 22.5 mm to (348.4, 80.4), turned to 0 degrees
- moved D1 3.54 mm to (78.0, 89.5)
- moved D10 3.54 mm to (344.5, 108.6)
- moved D11 3.54 mm to (325.6, 89.5)
- moved D14 3.54 mm to (323.0, 108.6)
- moved D15 3.54 mm to (306.6, 89.5)
- moved D17 3.54 mm to (182.5, 108.6)
- moved D19 3.54 mm to (287.5, 89.5)
- moved D22 3.54 mm to (258.7, 108.6)
- moved D29 3.54 mm to (125.3, 108.6)
- moved D32 3.54 mm to (97.0, 89.5)
- moved D34 3.54 mm to (363.6, 108.6)
- moved D37 3.54 mm to (277.7, 108.6)
- moved D8 3.54 mm to (211.3, 89.5)
- moved D9 3.54 mm to (220.6, 108.6)
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Routing:
- net /Row6: track 281.9 -> 250.8 mm
- net Net-(D4-Pad2): track 15.3 -> 24.9 mm
- net Net-(D47-Pad2): track 10.5 -> 17.1 mm
- net Net-(J1-Pad6): track 264.1 -> 269.8 mm
- net Net-(J1-Pad2): track 232.7 -> 238.1 mm
- net Net-(D62-Pad1): track 247.5 -> 242.9 mm
- net Net-(J1-Pad22): track 116.0 -> 112.9 mm
- net Net-(J1-Pad4): track 238.0 -> 235.7 mm
- net /Col5: track 447.3 -> 445.2 mm
- net Net-(D33-Pad1): track 165.1 -> 163.0 mm
- net /Col6: track 426.4 -> 424.3 mm
- net Net-(D63-Pad1): track 193.2 -> 191.1 mm
- net /Row3: track 343.2 -> 341.4 mm
- net Net-(D33-Pad2): track 180.4 -> 178.7 mm
- net /Row7: track 312.0 -> 311.1 mm
Other:
- outline, holes or cut-outs redrawn
- board text added: "Unified Keyboard Rev 1.10 http://osiweb.org"
- board text removed: "Unified Keyboard Rev 1.8 http://osiweb.org"

Commit message: Moved Cherry MX and futaba pads farther apart in combined footprint
- Offset cherry MX pads and aligners downward 0.004" from origin

- Offset futaba pads and aligners upward -0.004" from origin

- Update footprints in classic and sol-20 pcbs and aligners

- adjust mounting slots in Sol-20 aligners to match futaba or cherry offset
Other:
- board text added: "Unified Keyboard Rev 1.11 http://osiweb.org"
- board text removed: "Unified Keyboard Rev 1.10 http://osiweb.org"
