File: hardware/keyboard-sol/aligner-cherry/sol-aligner-cherry.kicad_pcb (KiCad board)
At the start: 2 copper layers, 386.1 x 116.3 mm, 88 parts, among them SW10 TAB: 1.25x, SW11 I, SW12 2, SW13 Zero, SW14 Q, SW15 O, SW16 3, SW17 Dash, SW18 W, SW19 P, SW20 4, SW21 Caret, SW22 E, SW23 AT, SW24 5, SW25 LT Bracket, SW26 R, SW27 Return: 1.5x, SW28 6, SW29 Backslash, SW30 T, SW31 Line Feed, SW32 7, SW33 RT Bracket, SW34 Y, SW35 Load, SW36 LT Ctrl, SW37 J, SW38 Upper Case: 1.5x, SW39 M, SW4 ESC: 1.75x, SW40 Shift Lock: 1.5x, SW41 K, SW42 LT Shift: 1.5x, SW43 Comma, SW44 A, SW45 L, SW46 Z, SW47 Period, SW48 S, SW49 Semicolon, SW5 8, SW50 X, SW51 Slash, SW52 D, SW53 Colon, SW54 C, SW55 RT Shift: 2x, SW56 F, SW57 DEL, SW58 V, SW59 Mode Select: 1.75x, SW6 BREAK, SW60 G, SW61 Repeat: 1.25x, SW62 B, SW63 H, SW64 RT Ctrl, SW65 N, SW66 Local, SW67 NP Dash, SW68 NP 4, SW69 NP Zero, SW7 U, SW70 Up Arrow, SW71 NP 7, SW72 NP 1, SW73 NP period, SW74 LT Arrow, SW75 NP asterisk, SW76 NP 5, SW77 NP plus, SW78 Spacebar, SW79 NP 8, SW8 1, SW80 NP 2, SW81 RT Arrow, SW82 NP divide, SW83 NP 6, SW84 Down Arrow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

Commit message: Replace wrong cherry aligner file.
Other:
- board text removed: "SOL-20 Cherry aligner. rev 1.0"
- board text removed: "Unified Keyboard https://github.com/osiweb/unified_retro_keyboard"
Changed lines of the file:
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@@
   (general
     (thickness 1.6)
-    (drawings 11)
+    (drawings 9)
     (tracks 0)
     (zones 0)
@@
     (pad "" np_thru_hole circle (at 0 0) (size 3.81 3.81) (drill 3.81) (layers *.Cu *.Mask))
   )
-  (gr_text "SOL-20 Cherry aligner.  rev 1.0" (at 182.118 111.6584) (layer F.SilkS)
-    (effects (font (size 2.032 2.032) (thickness 0.2032)))
-  )
-  (gr_text "Unified Keyboard    https://github.com/osiweb/unified_retro_keyboard" (at 370.713 112.014) (layer F.SilkS)
-    (effects (font (size 2.032 2.032) (thickness 0.2032)))
-  )
   (gr_circle (center 103.1875 206.7706) (end 105.7075 206.7706) (layer Edge.Cuts) (width 0.05))

Commit message: Add silk screen information to cherry aligner.
Other:
- board text added: "SOL-20 keyboard cherry MX aligner, rev 1.0"
- board text added: "Unified Keyboard Project https://github.com/osiweb/unified_retro_keyboard"
Changed lines of the file:
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@@
   (general
     (thickness 1.6)
-    (drawings 9)
+    (drawings 11)
     (tracks 0)
     (zones 0)
@@
     (pad "" np_thru_hole circle (at 0 0) (size 3.81 3.81) (drill 3.81) (layers *.Cu *.Mask))
   )
+  (gr_text "Unified Keyboard Project    https://github.com/osiweb/unified_retro_keyboard" (at 311.7088 114.4016) (layer F.SilkS)
+    (effects (font (size 2.032 2.032) (thickness 0.2032)) (justify left))
+  )
+  (gr_text "SOL-20 keyboard cherry MX aligner, rev 1.0" (at 141.6304 114.0206) (layer F.SilkS)
+    (effects (font (size 2.032 2.032) (thickness 0.2032)) (justify left))
+  )
   (gr_circle (center 103.1875 206.7706) (end 105.7075 206.7706) (layer Edge.Cuts) (width 0.05))
