File: hardware/keyboard-sol/kbd-sol.kicad_pcb (KiCad board)
At the start: 2 copper layers, 428.6 x 134.1 mm, 178 parts, among them J1 Controller, SW10 TAB: 1.25x, SW11 I, SW12 2, SW13 Zero, SW14 Q, SW15 O, SW16 3, SW17 Dash, SW18 W, SW19 P, SW20 4, SW21 Caret, SW22 E, SW23 AT, SW24 5, SW25 LT Bracket, SW26 R, SW27 Return: 1.5x, SW28 6, SW29 Backslash, SW30 T, SW31 Line Feed, SW32 7, SW33 RT Bracket, SW34 Y, SW35 Load, SW36 LT Ctrl, SW37 J, SW38 Upper Case: 1.5x, SW39 M, SW4 ESC: 1.75x, SW40 Shift Lock: 1.5x, SW41 K, SW42 LT Shift: 1.5x, SW43 Comma, SW44 A, SW45 L, SW46 Z, SW47 Period, SW48 S, SW49 Semicolon, SW5 8, SW50 X, SW51 Slash, SW52 D, SW53 Colon, SW54 C, SW55 RT Shift: 2x, SW56 F, SW57 DEL, SW58 V, SW59 Mode Select: 1.75x, SW6 BREAK, SW60 G, SW61 Repeat: 1.25x, SW62 B, SW63 H, SW64 RT Ctrl, SW65 N, SW66 Local, SW67 NP Dash, SW68 NP 4, SW69 NP Zero, SW7 U, SW70 Up Arrow, SW71 NP 7, SW72 NP 1, SW73 NP period, SW74 LT Arrow, SW75 NP asterisk, SW76 NP 5, SW77 NP plus, SW78 Spacebar, SW79 NP 8, SW8 1, SW80 NP 2, SW81 RT Arrow, SW82 NP divide, SW83 NP 6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

Commit message: Moved connector to top of board
Reduces required extra space at bottom of board.  Needed to fit in case.
Parts:
- moved J1 182.6 mm to (223.2, 68.3), turned to 270 degrees
Routing:
- net /Row6: track 604.6 -> 203.5 mm
- net /Row4: track 552.2 -> 184.2 mm
- net /Row11: track 82.6 -> 388.9 mm, vias 0 -> 1
- net /Row10: track 177.9 -> 433.5 mm, vias 0 -> 1
- net Net-(D88-Pad2): track 411.6 -> 191.1 mm
- net Net-(D88-Pad1): track 409.3 -> 192.3 mm
- net /Row8: track 420.5 -> 613.7 mm, vias 2 -> 1
- net /Row3: track 229.8 -> 395.3 mm, vias 2 -> 4
- net /Row9: track 217.1 -> 330.8 mm, vias 0 -> 1
- net Net-(D86-Pad2): track 348.6 -> 256.5 mm
- net Net-(D86-Pad1): track 349.4 -> 258.2 mm
- net Net-(D87-Pad1): track 342.3 -> 261.2 mm
- net Net-(D87-Pad2): track 340.5 -> 261.1 mm
- net /Row5: track 290.4 -> 213.4 mm, vias 1 -> 2
- net /Row1: track 326.6 -> 395.7 mm, vias 2 -> 3
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Other:
- outline, holes or cut-outs redrawn

Commit message: SOL keyboard adjustments
- Fixed position offset error in first three rows of the SOL keyboard

- moved key matrix interface connector to bottom of board so the parallel output
connector can be at the top of the keyboard.

- Adjusted size of mounting slots to accommodate #6 screws.

- ongoing clean up of traces.
Parts:
- removed the REF** at (263.6, 159.0)
- removed the REF** at (263.6, 174.3)
- removed Stabilizer (x2): MountingHole_3.5mm, MountingHole:MountingHole_3.5mm
- added REF**: mounting hole #6, MountingHole:MountingHole_4mm_Pad, F.Cu at (67.4, 73.9)
- added REF**: mounting hole #6, MountingHole:MountingHole_4mm_Pad, F.Cu at (405.8, 73.9)
- added REF**: mounting hole #6, MountingHole:MountingHole_4mm_Pad, F.Cu at (236.6, 73.9)
- J1: footprint unikbd:kbd_header_and_mounting_holes -> unikbd:kbd_header_two_mounting_holes
- SW78: footprint unikbd:Key_MX -> unikbd:Key_MX_Spacebar_5.25
- moved J1 131.8 mm to (137.2, 168.2), turned to 90 degrees
- moved D14 4.76 mm to (287.4, 86.2)
- moved D42 4.76 mm to (263.6, 124.3)
- moved SW23 4.76 mm to (287.4, 108.8)
- moved SW27 4.76 mm to (311.2, 108.8)
- moved SW29 4.76 mm to (335.1, 89.8)
- moved SW31 4.76 mm to (335.1, 108.8)
- moved SW57 4.76 mm to (311.2, 127.9)
- moved D12 4.76 mm to (258.8, 105.3)
- moved D21 4.76 mm to (173.1, 86.2)
- moved D23 4.76 mm to (163.5, 105.3)
- moved D27 4.76 mm to (182.6, 105.3)
- moved D29 4.76 mm to (211.2, 86.2)
- moved D38 4.76 mm to (244.6, 124.3)
- moved D49 4.76 mm to (149.3, 124.3)
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Connections:
- D63 pad 1: /Row8 -> /Row9
- D64 pad 1: /Row9 -> /Row10
- D65 pad 1: /Row10 -> /Row11
- D66 pad 1: /Row11 -> /Row12
- D67 pad 1: /Row8 -> /Row9
- D68 pad 1: /Row9 -> /Row10
- D69 pad 1: /Row10 -> /Row11
- D70 pad 1: /Row11 -> /Row12
- D71 pad 1: /Row8 -> /Row9
- D72 pad 1: /Row9 -> /Row10
- D73 pad 1: /Row10 -> /Row11
- D74 pad 1: /Row11 -> /Row12
- D75 pad 1: /Row8 -> /Row9
- D76 pad 1: /Row9 -> /Row10
- D77 pad 1: /Row10 -> /Row11
- D78 pad 1: /Row8 -> /Row9
- D79 pad 1: /Row9 -> /Row10
- D80 pad 1: /Row10 -> /Row11
- D81 pad 1: /Row8 -> /Row9
- D82 pad 1: /Row9 -> /Row10
- D83 pad 1: /Row10 -> /Row11
- D84 pad 1: /Row8 -> /Row9
- D85 pad 1: /Row8 -> /Row9
Routing:
- net /Row8: track 613.7 -> 0.00 mm, vias 1 -> 0
- net /Row12: track 0.00 -> 265.1 mm
- net /Row5: track 213.4 -> 476.5 mm
- net /Row7: track 215.7 -> 448.6 mm
- net /Row4: track 184.2 -> 416.3 mm, vias 1 -> 0
- net /Row2: track 408.6 -> 238.7 mm, vias 1 -> 2
- net /Row3: track 395.3 -> 240.0 mm, vias 4 -> 3
- net /Col6: track 465.7 -> 614.7 mm
- net Net-(D87-Pad2): track 261.1 -> 115.3 mm
- net Net-(D87-Pad1): track 261.2 -> 116.1 mm
- net Net-(D86-Pad1): track 258.2 -> 124.1 mm
- net Net-(D86-Pad2): track 256.5 -> 122.7 mm
- net /Row0: track 368.9 -> 247.0 mm, vias 1 -> 2
- net /Col3: track 754.5 -> 659.2 mm, vias 0 -> 2
- net /Col0: track 667.5 -> 757.9 mm, vias 1 -> 0
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Other:
- board size 428.6 x 134.1 mm -> 428.6 x 116.3 mm
- board text added: "Key spacing guide: Vertical: 0.75 inch. Key1, Key2 -> Centers (inches) 1.00, 1.00 -> 0.75 1.00, 1.25 -> 0.84375 1.00, 1.50 -> 0.9375 1.00, 1.75 -> 1.03125 1.00, 2.00 -> 1.125 1.25, 1.25 -> 0.9375 1.25, 1.50 -> 1.03125 1.25, 2.00 -> 1.21875 1.50, 1.50 -> 1.125 1.50, 2.00 -> 1.3125 1.75, 2.00. ->. 1.40625 8.00, 1.00 -> 3.375 8.00, 1.25 -> 3.46875 8.00, 1.50 -> 3.5625"
- board text removed: "Key spacing guide: Vertical: 0.75 inch. Key1, Key2 -> Centers (inches) 1.00, 1.00 -> 0.75 1.00, 1.25 -> 0.84375 1.00, 1.50 -> 0.9375 1.00, 1.75 -> 1.03125 1.00, 2.00 -> 1.125 1.25, 1.25 -> 0.9375 1.25, 1.50 -> 1.03125 1.25, 2.00 -> 1.21875 1.50, 1.50 -> 1.125 1.50, 2.00 -> 1.3125 8.00, 1.00 -> 3.375 8.00, 1.25 -> 3.46875 8.00, 1.50 -> 3.5625"

Commit message: Add Cherry and Futaba aligners and add text to PCB
Parts:
- moved D18 68.1 mm to (361.0, 127.0)
- moved D46 68.1 mm to (337.2, 165.1)
- moved D58 68.1 mm to (396.7, 165.1)
- moved D74 68.1 mm to (480.1, 203.2)
- moved D79 68.1 mm to (480.1, 127.0)
- moved D80 68.1 mm to (480.1, 165.1)
- moved D82 68.1 mm to (480.1, 146.1)
- moved D85 68.1 mm to (420.5, 203.2)
- moved SW35 68.1 mm to (408.6, 149.6)
- moved SW64 68.1 mm to (408.6, 168.7)
- moved SW68 68.1 mm to (432.4, 168.7)
- moved SW69 68.1 mm to (432.4, 206.8)
- moved SW71 68.1 mm to (432.4, 149.6)
- moved SW88 68.1 mm to (408.6, 206.8)
- moved D83 68.1 mm to (480.1, 184.2)
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Other:
- outline, holes or cut-outs redrawn
- board text added: "SOL-20 keyboard rev 1.0"
- board text added: "Unified Keyboard Project. https://github.com/osiweb/unified_retro_keyboard"

Commit message: Added aligners for SOL keyboard
- options for complete aligner, and split main/numpad aligners
- adjusted aligner spacer mounting holes on PCB.
Parts:
- removed the REF** at (121.9, 114.7)
- removed the REF** at (460.3, 114.7)
- removed the REF** at (291.1, 114.7)
- added REF**: MountingHole_3.2mm_M3, MountingHole:MountingHole_3.2mm_M3, F.Cu at (113.3, 219.5)
- added REF**: MountingHole_3.2mm_M3, MountingHole:MountingHole_3.2mm_M3, F.Cu at (408.6, 219.5)
- added REF**: MountingHole_3.2mm_M3, MountingHole:MountingHole_3.2mm_M3, F.Cu at (470.5, 219.5)
- added REF**: MountingHole_3.2mm_M3, MountingHole:MountingHole_3.2mm_M3, F.Cu at (432.4, 219.5)
- added REF**: MountingHole_3.2mm_M3, MountingHole:MountingHole_3.2mm_M3, F.Cu at (470.5, 114.1)
- added REF**: MountingHole_3.2mm_M3, MountingHole:MountingHole_3.2mm_M3, F.Cu at (432.4, 114.1)
- added REF**: MountingHole_3.2mm_M3, MountingHole:MountingHole_3.2mm_M3, F.Cu at (408.6, 114.0)
- added REF**: MountingHole_3.2mm_M3, MountingHole:MountingHole_3.2mm_M3, F.Cu at (115.7, 114.0)
- added REF**: MountingHole_3.2mm_M3, MountingHole:MountingHole_3.2mm_M3, F.Cu at (262.2, 114.0)
Routing:
- net /Row12: track 265.1 -> 269.9 mm
- net /Row5: track 476.5 -> 479.8 mm
- net /Row11: track 400.3 -> 403.4 mm
- net Net-(D88-Pad1): track 192.8 -> 190.7 mm
- net /Row4: track 416.3 -> 414.2 mm
- net Net-(D88-Pad2): track 190.4 -> 188.3 mm
- net Net-(D87-Pad1): track 116.1 -> 114.0 mm
- net Net-(D86-Pad1): track 124.1 -> 122.0 mm
- net Net-(D87-Pad2): track 115.3 -> 113.2 mm
- net Net-(D86-Pad2): track 122.7 -> 120.6 mm
- net /Row10: track 440.5 -> 441.3 mm
Other:
- board size 428.6 x 116.3 mm -> 428.6 x 117.7 mm

Commit message: Add series resistors to LEDs and stabilizer to 2u shift
Parts:
- added R1: 470, Resistor_THT:R_Axial_DIN0207_L6.3mm_D2.5mm_P10.16mm_Horizontal, F.Cu at (94.0, 195.4)
- added R2: 470, Resistor_THT:R_Axial_DIN0207_L6.3mm_D2.5mm_P10.16mm_Horizontal, F.Cu at (94.1, 218.0)
- added R3: 470, Resistor_THT:R_Axial_DIN0207_L6.3mm_D2.5mm_P10.16mm_Horizontal, F.Cu at (94.1, 180.9)
- SW55: footprint unikbd:Key_MX -> unikbd:Key_MX_2u
- moved D52 8.61 mm to (384.3, 184.2)
- moved D64 4.64 mm to (446.7, 127.0)
- moved D65 4.64 mm to (446.7, 165.1)
- moved D66 4.64 mm to (446.7, 203.2)
- moved D68 4.64 mm to (446.7, 146.1)
- moved D69 4.64 mm to (446.7, 184.2)
- moved SW73 4.64 mm to (456.1, 206.8)
- moved SW75 4.64 mm to (456.1, 130.6)
- moved SW76 4.64 mm to (456.1, 168.7)
- moved SW79 4.64 mm to (456.1, 149.6)
- moved SW80 4.64 mm to (456.1, 187.7)
- moved D70 4.64 mm to (465.6, 203.2)
- moved D72 4.64 mm to (465.6, 127.0)
- moved D73 4.64 mm to (465.6, 165.1)
- moved D74 4.64 mm to (484.7, 203.2)
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Connections:
- J1 pad 16: Net-(D87-Pad1) -> Net-(J1-Pad16)
- J1 pad 24: Net-(D88-Pad1) -> Net-(J1-Pad24)
- J1 pad 8: Net-(D86-Pad1) -> Net-(J1-Pad8)
Routing:
- net Net-(J1-Pad24): track 0.00 -> 167.3 mm, vias 0 -> 1
- net Net-(D88-Pad1): track 190.7 -> 42.6 mm, vias 1 -> 2
- net Net-(J1-Pad16): track 0.00 -> 122.8 mm, vias 0 -> 1
- net Net-(J1-Pad8): track 0.00 -> 122.0 mm, vias 0 -> 1
- net Net-(D86-Pad1): track 122.0 -> 13.5 mm
- net Net-(D87-Pad1): track 114.0 -> 11.9 mm
- net /Col0: track 757.9 -> 776.5 mm
- net /Col5: track 718.3 -> 734.7 mm
- net /Row3: track 240.0 -> 253.1 mm
- net Net-(D52-Pad2): track 9.50 -> 18.1 mm
- net /Col2: track 809.5 -> 814.3 mm
- net /Col3: track 659.2 -> 663.9 mm
- net /Row12: track 269.9 -> 274.5 mm
- net /Col1: track 805.0 -> 809.6 mm
- net /Row10: track 441.3 -> 445.9 mm
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Other:
- board text added: "SOL-20 keyboard rev 1.1"
- board text removed: "SOL-20 keyboard rev 1.0"

Commit message: Moved mounting slots from keyboard PCB to aligners
- This allows the PCB to sink below the mounting brackets.  The aligner height can
be adjusted relative to the mounting brackets using spacers.

- changed futaba aligners to use cherry stabilizers.

- bumped rev number
Parts:
- moved R2 7.14 mm to (96.4, 211.3)
- moved R1 2.44 mm to (96.4, 195.4)
- moved R3 2.34 mm to (96.4, 180.9)
- renumbered D86 to LED1, D87 to LED2, D88 to LED3
Routing:
- net Net-(J1-Pad24): track 167.3 -> 161.7 mm
- net Net-(J1-Pad22): track 188.3 -> 183.1 mm
- net Net-(J1-Pad16): track 122.8 -> 118.8 mm
- net /Row4: track 414.2 -> 410.3 mm
- net Net-(J1-Pad8): track 122.0 -> 119.6 mm
- net /Row10: track 445.9 -> 443.7 mm, vias 1 -> 0
- net /Col5: track 734.7 -> 733.2 mm
- net Net-(LED3-Pad1): track 42.6 -> 41.8 mm
- net Net-(LED2-Pad1): track 11.9 -> 12.7 mm
- net Net-(LED1-Pad1): track 13.5 -> 12.8 mm
Other:
- board size 428.6 x 117.7 mm -> 396.2 x 117.7 mm

Commit message: Minor cleanups
Connections:
- net /Row13 renamed Net-(J1-Pad37)
- net /Row14 renamed Net-(J1-Pad35)
- net /Row15 renamed Net-(J1-Pad33)
- net /Row8 renamed Net-(J1-Pad34)
Routing:
- net /Col2: track 814.3 -> 813.2 mm
Other:
- board text added: "SOL-20 keyboard rev 1.4"
- board text removed: "SOL-20 keyboard rev 1.1"

Commit message: Adjsut mounting slots and alignment of mounting holes.
Parts:
- moved REF** 5.95 mm to (256.2, 114.1)
- moved REF** 0.09 mm to (408.6, 114.1)
- moved REF** 0.09 mm to (115.7, 114.1)
Changed lines of the file:
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@@
   )
   (module MountingHole:MountingHole_3.2mm_M3 locked (layer F.Cu)
-    (at 408.61488 113.9952)
+    (at 408.61488 114.08156)
     (descr "Mounting Hole 3.2mm, no annular, M3")
     (tags "mounting hole 3.2mm no annular m3")
@@
   )
   (module MountingHole:MountingHole_3.2mm_M3 locked (layer F.Cu)
-    (at 115.72113 113.9952)
+    (at 115.72113 114.08156)
     (descr "Mounting Hole 3.2mm, no annular, M3")
     (tags "mounting hole 3.2mm no annular m3")
@@
   )
   (module MountingHole:MountingHole_3.2mm_M3 locked (layer F.Cu)
-    (at 262.168005 113.9952)
+    (at 256.21488 114.08156)
     (descr "Mounting Hole 3.2mm, no annular, M3")
     (tags "mounting hole 3.2mm no annular m3")
