File: hardware/keyboard-sol/aligner-futaba/aligner-futaba-numpad.kicad_pcb (KiCad board)
At the start: 2 copper layers, 62.1 x 116.9 mm, 19 parts, among them SW67 NP Dash, SW68 NP 4, SW69 NP Zero, SW71 NP 7, SW72 NP 1, SW73 NP period, SW75 NP asterisk, SW76 NP 5, SW77 NP plus, SW79 NP 8, SW80 NP 2, SW82 NP divide, SW83 NP 6, SW85 NP 9, SW86 NP 3

Commit message: Moved mounting slots from keyboard PCB to aligners
- This allows the PCB to sink below the mounting brackets.  The aligner height can
be adjusted relative to the mounting brackets using spacers.

- changed futaba aligners to use cherry stabilizers.

- bumped rev number
Parts:
- removed the REF** at (187.9, 219.3)
- removed the REF** at (149.8, 219.3)
- removed the REF** at (187.9, 113.9)
- removed the REF** at (149.8, 113.9)
- added REF**: MountingHole_3.2mm_M3, MountingHole:MountingHole_3.2mm_M3, F.Cu at (432.4, 219.5)
- added REF**: MountingHole_3.2mm_M3, MountingHole:MountingHole_3.2mm_M3, F.Cu at (470.5, 219.5)
- added REF**: MountingHole_3.2mm_M3, MountingHole:MountingHole_3.2mm_M3, F.Cu at (470.5, 114.1)
- added REF**: MountingHole_3.2mm_M3, MountingHole:MountingHole_3.2mm_M3, F.Cu at (432.4, 114.1)
- moved SW67 282.6 mm to (432.4, 130.6)
- moved SW68 282.6 mm to (432.4, 168.7)
- moved SW69 282.6 mm to (432.4, 206.8)
- moved SW71 282.6 mm to (432.4, 149.6)
- moved SW72 282.6 mm to (432.4, 187.7)
- moved SW77 282.6 mm to (470.5, 206.8)
- moved SW82 282.6 mm to (470.5, 130.6)
- moved SW83 282.6 mm to (470.5, 168.7)
- moved SW85 282.6 mm to (470.5, 149.6)
- moved SW86 282.6 mm to (470.5, 187.7)
- moved SW73 282.6 mm to (451.5, 206.8)
- moved SW75 282.6 mm to (451.5, 130.6)
- moved SW76 282.6 mm to (451.5, 168.7)
- moved SW79 282.6 mm to (451.5, 149.6)
- moved SW80 282.6 mm to (451.5, 187.7)
Other:
- board size 62.1 x 116.9 mm -> 83.7 x 117.7 mm
- board text added: "SOL-20 Futaba aligner (numpad) Rev 1.1"
- board text added: "https://github.com/osiweb/unified_retro_keyboard Unified Keyboard Project"
- board text removed: "SOL-20 Futaba MD-4PCS aligner (NumPad) Rev 1.0"
- board text removed: "https://github.com/osiweb/unified_retro_keyboard"

Commit message: Adjsut mounting slots and alignment of mounting holes.
Other:
- outline, holes or cut-outs redrawn
- board text added: "SOL-20 Futaba aligner (numpad) Rev 1.4"
- board text removed: "SOL-20 Futaba aligner (numpad) Rev 1.1"
Changed lines of the file:
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@@
     (pad 1 np_thru_hole circle (at 0 0) (size 3.2 3.2) (drill 3.2) (layers *.Cu *.Mask))
   )
-  (gr_line (start 505.44984 200.12914) (end 505.44984 134.08914) (layer Edge.Cuts) (width 0.1016))
+  (gr_line (start 505.44984 202.66914) (end 505.44984 136.62914) (layer Edge.Cuts) (width 0.1016))
   (gr_line (start 421.767 224.79) (end 421.767 107.0864) (layer Edge.Cuts) (width 0.1016))
-  (gr_text "SOL-20 Futaba aligner  (numpad)\nRev 1.1\n" (at 500.2784 193.6496 90) (layer F.SilkS)
+  (gr_text "SOL-20 Futaba aligner  (numpad)\nRev 1.4\n" (at 500.2784 196.1896 90) (layer F.SilkS)
     (effects (font (size 2.032 2.032) (thickness 0.2032)) (justify left))
   )
@@
     (effects (font (size 2.032 2.032) (thickness 0.3048)) (justify left))
   )
-  (gr_line (start 505.45238 107.0864) (end 505.45238 130.27914) (layer Edge.Cuts) (width 0.1016))
-  (gr_line (start 505.45238 224.79) (end 505.45238 203.93914) (layer Edge.Cuts) (width 0.1016))
-  (gr_line (start 488.78109 203.93914) (end 505.44984 203.93914) (layer Edge.Cuts) (width 0.1016))
-  (gr_line (start 488.78109 134.08914) (end 505.44984 134.08914) (layer Edge.Cuts) (width 0.1016))
-  (gr_line (start 488.78109 130.27914) (end 505.44984 130.27914) (layer Edge.Cuts) (width 0.1016))
-  (gr_arc (start 488.78109 132.18414) (end 488.78109 130.27914) (angle -180) (layer Edge.Cuts) (width 0.1016))
-  (gr_line (start 488.78109 200.12914) (end 505.44984 200.12914) (layer Edge.Cuts) (width 0.1016))
-  (gr_arc (start 488.78109 202.03414) (end 488.78109 200.12914) (angle -180) (layer Edge.Cuts) (width 0.1016))
+  (gr_line (start 505.45238 107.0864) (end 505.45238 132.81914) (layer Edge.Cuts) (width 0.1016))
+  (gr_line (start 505.45238 224.79) (end 505.45238 206.47914) (layer Edge.Cuts) (width 0.1016))
+  (gr_line (start 488.78109 206.47914) (end 505.44984 206.47914) (layer Edge.Cuts) (width 0.1016))
+  (gr_line (start 488.78109 136.62914) (end 505.44984 136.62914) (layer Edge.Cuts) (width 0.1016))
+  (gr_line (start 488.78109 132.81914) (end 505.44984 132.81914) (layer Edge.Cuts) (width 0.1016))
+  (gr_arc (start 488.78109 134.72414) (end 488.78109 132.81914) (angle -180) (layer Edge.Cuts) (width 0.1016))
+  (gr_line (start 488.78109 202.66914) (end 505.44984 202.66914) (layer Edge.Cuts) (width 0.1016))
+  (gr_arc (start 488.78109 204.57414) (end 488.78109 202.66914) (angle -180) (layer Edge.Cuts) (width 0.1016))
   (gr_line (start 421.767 224.79) (end 505.45238 224.79) (layer Edge.Cuts) (width 0.1))
   (gr_line (start 505.45238 107.0864) (end 421.767 107.0864) (layer Edge.Cuts) (width 0.1016))
