File: hardware/keyboard-sol/aligner-futaba/aligner-futaba.kicad_pcb (KiCad board)
At the start: 2 copper layers, 428.6 x 117.7 mm, 108 parts, among them SW10 TAB: 1.25x, SW11 I, SW12 2, SW13 Zero, SW14 Q, SW15 O, SW16 3, SW17 Dash, SW18 W, SW19 P, SW20 4, SW21 Caret, SW22 E, SW23 AT, SW24 5, SW25 LT Bracket, SW26 R, SW27 Return: 1.5x, SW28 6, SW29 Backslash, SW30 T, SW31 Line Feed, SW32 7, SW33 RT Bracket, SW34 Y, SW35 Load, SW36 LT Ctrl, SW37 J, SW38 Upper Case: 1.5x, SW39 M, SW4 ESC: 1.75x, SW40 Shift Lock: 1.5x, SW41 K, SW42 LT Shift: 1.5x, SW43 Comma, SW44 A, SW45 L, SW46 Z, SW47 Period, SW48 S, SW49 Semicolon, SW5 8, SW50 X, SW51 Slash, SW52 D, SW53 Colon, SW54 C, SW55 RT Shift: 2x, SW56 F, SW57 DEL, SW58 V, SW59 Mode Select: 1.75x, SW6 BREAK, SW60 G, SW61 Repeat: 1.25x, SW62 B, SW63 H, SW64 RT Ctrl, SW65 N, SW66 Local, SW67 NP Dash, SW68 NP 4, SW69 NP Zero, SW7 U, SW70 Up Arrow, SW71 NP 7, SW72 NP 1, SW73 NP period, SW74 LT Arrow, SW75 NP asterisk, SW76 NP 5, SW77 NP plus, SW78 Spacebar, SW79 NP 8, SW8 1, SW80 NP 2, SW81 RT Arrow, SW82 NP divide, SW83 NP 6, SW84 Down Arrow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

Commit message: Update Sol-20 keyboard to use fixed footprints
- Update all footprints on sol-20 keyboard and aligners

- Add soldermask clearance around cherry MX posts

- Move Cherry MX pads down 1 mil, and Futaba pads up 2 mils

- Adjust Cherry aligner footprints down 1 mil

- Adjust Futaba aligner footprints up 2 mils

- Move mounting slots up 1 mil on Cherry aligner

- Move mounting slots down 1 mil on Futaba aligner

- incorporate improved stabilizer post adapters in futaba aligner

- add slots for stabilizer posts in futaba aligner and Sol kebyoard PCB

- Move stabilizer bar bend guide to left bottom edge to facilitate bending

- Bump rev to 1.6
Parts:
- removed the REF** at (87.0, 165.2)
- removed the REF** at (495.2, 167.2)
- removed the REF** at (495.2, 169.5)
- removed the REF** at (495.2, 171.9)
- removed the REF** at (184.8, 220.9)
- removed the REF** at (87.0, 167.6)
- removed the REF** at (87.0, 169.9)
- removed the REF** at (289.0, 113.6)
- removed the REF** at (291.3, 113.6)
- removed the REF** at (293.7, 113.6)
- removed the REF** at (368.4, 113.7)
- removed the REF** at (370.7, 113.7)
- removed the REF** at (373.1, 113.7)
- added ?: , , F.Cu at (413.8, 5.21)
- added ?: , , F.Cu at (206.4, 194.8)
- added ?: , , F.Cu at (127.0, 194.6)
- added ?: , , F.Cu at (5.59, 3.30)
- moved REF** 108.0 mm to (210.2, 220.4)
Other:
- outline, holes or cut-outs redrawn
- board text added: "SOL-20 Futaba MD-4PCS aligner Rev 1.6"
- board text removed: "SOL-20 Futaba MD-4PCS aligner Rev 1.5"

Commit message: Include futaba pad/aligner shifts in futaba aligner
Parts:
- added ?: , , F.Cu at (300.9, 277.6)
- moved REF** 0.05 mm to (210.2, 220.3)
Other:
- outline, holes or cut-outs redrawn
- board text added: "SOL-20 Futaba MD-4PCS aligner Rev 1.7"
- board text removed: "SOL-20 Futaba MD-4PCS aligner Rev 1.6"
