File: hardware/interface-osi/interface-osi.kicad_pcb (KiCad board)
At the start: 2 copper layers, 124.5 x 132.1 mm, 79 parts, among them J1 KBD port, J2 Key Matrix, J3 Expansion, J4 Sound, J5 ~RESET~, U1 74LS138, U10 74HC14, U11 4066, U2 74LS04, U3 74HC240, U4 74HC240, U5 74LS373, U6 74LS373, U7 74LS193, U8 74LS193, U9 74LS390

Commit message: mechanical fit and buildability fixes
- Moved header slightly forward

- Moved interface mount holes do reduce interference with case mount holes

- For all keys in classic keyboard, add option for either through-hole or SMT
diodes and resistors.
Parts:
- J2: footprint unikbd:PinHeader_2x20_P2.54mm_Vertical -> unikbd:kbd_header_and_mounting_holes
- JP1: value S1 Select -> Jumper_3_Open
- moved D11 5.08 mm to (250.7, 81.2)
- moved D14 5.08 mm to (260.3, 81.2)
- moved D9 5.08 mm to (244.2, 81.2)
- moved R1 5.08 mm to (244.2, 84.0)
- moved R3 5.08 mm to (250.7, 84.0)
- moved R6 5.08 mm to (260.3, 84.0)
- moved D10 5.08 mm to (247.4, 81.2)
- moved D12 5.08 mm to (253.9, 81.2)
- moved D13 5.08 mm to (257.1, 81.2)
- moved D15 5.08 mm to (263.6, 81.2)
- moved D16 5.08 mm to (266.8, 81.2)
- moved R2 5.08 mm to (247.4, 84.0)
- moved R4 5.08 mm to (253.9, 84.0)
- moved R5 5.08 mm to (257.1, 84.0)
- moved R7 5.08 mm to (263.6, 84.0)
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Routing:
- net /Sound/S1: track 121.8 -> 129.8 mm
- net /Sound/S7: track 70.8 -> 78.1 mm
- net /Sound/S6: track 57.0 -> 63.3 mm, vias 2 -> 3
- net /Sound/S0: track 44.8 -> 49.9 mm
- net /Sound/S4: track 33.1 -> 35.9 mm
- net /D1: track 88.2 -> 85.6 mm
- net /~KBE: track 88.7 -> 91.1 mm
- net /~A1: track 88.0 -> 90.2 mm
- net /Sound/S2: track 35.1 -> 37.2 mm
- net /Sound/S5: track 50.3 -> 52.4 mm
- net Net-(C14-Pad2): track 35.9 -> 38.0 mm
- net /D3: track 97.2 -> 95.1 mm
- net /Sound/S3: track 40.8 -> 42.3 mm
- net /~A0: track 88.5 -> 89.9 mm
- net /D7: track 51.3 -> 49.9 mm
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Other:
- outline, holes or cut-outs redrawn
- board text added: "Unified Keyboard OSI Interface Rev 1.2"
- board text added: "Unified Keyboard OSO Interface Rev 1.2"
- board text removed: "Mounting holes: 0.125" Non-plated 2.5" square spacing Pin 1 of connector 0.31", 0" (x,y) relative to center of left lower hole."
- board text removed: "Pin 1 of keyboard connector must be at least 3.5" from pin 1 of interface connector in order for interface connector to be accessible with keyboard assembled."
- board text removed: "Unified Keyboard OSI Interface Rev 1.1"
- board text removed: "Unified Keyboard OSO Interface Rev 1.1"
