File: hardware/keyboard-classic/Aligner-cherry/aligner-cherry.kicad_pcb (KiCad board)
At the start: 2 copper layers, 307.3 x 103.9 mm, 72 parts, among them SW1 Clear, SW10 Bracket_Open, SW11 6, SW12 Y, SW13 Return, SW14 Dash, SW15 5, SW16 T, SW17 Line Feed, SW18 Colon, SW19 4, SW2 Repeat, SW20 R, SW21 O, SW22 0, SW23 3, SW24 E, SW25 L, SW26 9, SW27 2, SW28 W, SW29 Period, SW3 Tilde, SW30 8, SW31 1, SW32 Ampersand, SW33 Break, SW34 Rubout, SW35 R_Shift, SW36 P, SW37 Comma, SW38 K, SW39 L_Shift, SW4 I, SW40 Semicolon, SW41 M, SW42 J, SW43 Fwd_Slash, SW44 N, SW45 H, SW46 SPACE, SW47 B, SW48 G, SW49 ESC, SW5 Here_is, SW50 Z, SW51 V, SW52 F, SW53 CTRL, SW54 A, SW55 C, SW56 D, SW57 Backslash, SW58 Q, SW59 X, SW6 Bracket_Close, SW60 S, SW7 7, SW8 U, SW9 Shift_Lock

Commit message: OSI mounting holes
- Add OSI-compatible mounting holes.
- Adjust keyboard and aligner holes to make room for the OSI mounting holes
- Change "Universal Keyboard" to "Unified Keyboard" in the design files.
Parts:
- removed the REF** at (107.8, 171.4)
- removed the REF** at (363.2, 171.4)
- removed the REF** at (284.6, 171.4)
- added REF**: MountingHole_3.5mm, MountingHole:MountingHole_3.5mm, F.Cu at (102.7, 171.4)
- added REF**: MountingHole_3.5mm, MountingHole:MountingHole_3.5mm, F.Cu at (358.1, 171.4)
- added REF**: MountingHole_3.5mm, MountingHole:MountingHole_3.5mm, F.Cu at (289.7, 171.4)
Other:
- board text added: "Unified Keyboard Rev 1.2 http://osiweb.org Cherry Key Aligner"
- board text removed: "Universal Keyboard Rev 1.1 http://osiweb.org Cherry Key Aligner"

Commit message: Finalize layout and mounting
- Add apple 2 mounting slots (and stretch PCB to accommodate slots
- Add pass-through holes in aligners for OSI keyboard spacers
- Move 'ESC' key next to '1' key
- Add TAB key next to Q key
- remove 'here is' and finalize "helper" keys along left side of keyboard
- move legends off of PCB traces
- update to release 1.3
Parts:
- removed the REF** at (117.3, 163.3)
- added REF**: OSHW-Logo2_9.8x8mm_SilkScreen, Symbol:OSHW-Logo2_9.8x8mm_SilkScreen, F.Cu at (119.3, 174.2)
- added REF**: OSI mounting holes, unikbd:OSI_spacer_holes, F.Cu at (196.9, 166.0)
- added SW61: FN, unikbd:Cherry aligner, F.Cu at (82.8, 166.1)
- added SW62: ESC, unikbd:Cherry aligner, F.Cu at (68.6, 89.8)
- SW1: value Clear -> RT Arrow
- SW2: value Repeat -> LT Arrow
- SW32: value Ampersand -> @ (AT)
- SW49: value ESC -> TAB
- SW5: value Here_is -> Repeat
- SW9: value Shift_Lock -> Caps Lock
Other:
- board size 307.3 x 103.9 mm -> 312.4 x 114 mm
- board text added: "Unified Keyboard Rev 1.3 http://osiweb.org Cherry Key Aligner"
- board text removed: "Unified Keyboard Rev 1.2 http://osiweb.org Cherry Key Aligner"

Commit message: Keyboard layout updates
- Add extra key to the left side of row 4 to permit "inverted T" for those who
  want it.

- Tiny shifts of several keys to correct key distances

- Include mounting holes with daughter board connector, to ensure consistency.
Parts:
- moved SW12 0.28 mm to (192.4, 108.8)
- moved SW17 0.28 mm to (287.6, 108.8)
- moved SW20 0.28 mm to (154.3, 108.8)
- moved SW22 0.28 mm to (249.5, 108.8)
- moved SW36 0.28 mm to (268.6, 108.8)
- moved SW8 0.28 mm to (211.4, 108.8)
- moved SW28 0.28 mm to (116.2, 108.8)
- moved SW58 0.28 mm to (97.1, 108.8)
- moved SW16 0.28 mm to (173.3, 108.8)
- moved SW24 0.28 mm to (135.2, 108.8)
- moved SW4 0.28 mm to (230.5, 108.8)
- moved SW13 0.24 mm to (311.5, 108.8)
- moved REF** 0.22 mm to (197.2, 166.0)
- moved SW46 0.22 mm to (197.2, 166.0)
- moved SW39 0.15 mm to (87.6, 146.9)
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Other:
- board text added: "Distances: Vertical: 0.75 inch Horizontal (1x - 1x): 0.75 inch Horizontal (1x - 1.5x): 0.975 inch Horizontal (Row 1 left key -> Row 2 left key): 0.375 inch Horizontal (Row 2 left key -> Row 3 left key): 0.1875 inch Horizontal (Row 3 left key -> Row 4 left key): 0.1875 inch Horizontal (Row 4 left key -> Row 5 left key): -0.1875 inch Horizontal (Row 5 left key -> space bar): 4.5 inch"
- board text added: "Unified Keyboard Rev 1.4 http://osiweb.org Cherry Key Aligner"
- board text removed: "Distances: Vertical: 0.75 inch Horizontal (1x - 1x): 0.75 inch Horizontal (1x - 1.5x): 0.939 inch Horizontal (Row 1 left key -> Row 2 left key): -0.379 inch Horizontal (Row 2 left key -> Row 3 left key): 0.187 inch Horizontal (Row 3 left key -> Row 4 left key): 0.186 inch Horizontal (Row 4 left key -> space bar): 4.310 inch"
- board text removed: "Unified Keyboard Rev 1.3 http://osiweb.org Cherry Key Aligner"

Commit message: Multiple fixes to classic keyboard for fit and build ease
- remove material from PCB to allow keyboard to fit in Apple II case

- enlarge center hole on cherry MX footprints slightly, to 0.160" to allow
slightly more tolerance, which eases assembly.

- include holes for LEDs on futaba aligner

- include extra pads on main PCB for LEDs with futaba keys

- Add LED on LINE FEED which maps to REPEAT/CAPSLOCK on Apple II keymap
Parts:
- added ?: , , F.Cu at (98.9, 189.5)
- added REF**: LED, MountingHole:MountingHole_3.2mm_M3, F.Cu at (364.8, 127.9)
- added REF**: LED, MountingHole:MountingHole_3.2mm_M3, F.Cu at (292.4, 137.0)
- added REF**: LED Hole, MountingHole:MountingHole_3.2mm_M3, F.Cu at (93.0, 190.9)
- renumbered REF** to SW46
Routing:
- net (no net): vias 0 -> 1
Other:
- outline, holes or cut-outs redrawn
- board text added: "Unified Keyboard Rev 1.6 http://osiweb.org Cherry Key Aligner"
- board text removed: "Unified Keyboard Rev 1.4 http://osiweb.org Cherry Key Aligner"

Commit message: Fixes for classic keyboard outline and mounting hole patters
- Adjust upper right corner circular cutout for AppleII+ case fit.

- Adjust OSI mounting hole pattern for improved fit.

- Changed OSI mount holes along top of keyboard to slots, to fit both C2P (542
keyboard) and C4P (542 Rev B/c keyboards).

- PCB and aligners must be slightly taller to accommodate the slots along the
top row
Parts:
- removed ?: , 
- removed the REF** at (364.8, 127.9)
- removed the REF** at (292.4, 137.0)
- removed the REF** at (93.0, 190.9)
- removed the SW46 at (197.2, 166.0)
- added REF**: OSI mounting holes, unikbd:OSI_spacer_holes, F.Cu at (197.2, 166.0)
- added REF**: MountingHole_2.1mm, MountingHole:MountingHole_2.1mm, F.Cu at (263.7, 177.4)
- added REF**: MountingHole_2.1mm, MountingHole:MountingHole_2.1mm, F.Cu at (130.3, 177.4)
- SW1, SW10, SW11, SW12, SW13, SW14, SW15, SW16, SW17, SW18, SW19, SW2, SW20, SW21, SW22, SW23, SW24, SW25, SW26, SW27, SW28, SW29, SW3, SW30, SW31, SW32, SW33, SW34, SW35, SW36, SW37, SW38, SW39, SW4, SW40, SW41, SW42, SW43, SW44, SW45, SW47, SW48, SW49, SW5, SW50, SW51, SW52, SW53, SW54, SW55, SW56, SW57, SW58, SW59, SW6, SW60, SW61, SW62, SW7, SW8, SW9: footprint unikbd:Cherry aligner -> unikbd:Key_MX_Aligner
Routing:
- net (no net): vias 1 -> 0
Other:
- board size 312.4 x 114 mm -> 312.4 x 118.1 mm
- board text added: "Stabilizer bend guide"
- board text added: "Stabilzer bend guide"
- board text added: "Unified Keyboard Rev 1.7 http://osiweb.org Cherry Key Aligner"
- board text removed: "Unified Keyboard Rev 1.6 http://osiweb.org Cherry Key Aligner"

Commit message: mechanical fit and buildability fixes
- Moved header slightly forward

- Moved interface mount holes do reduce interference with case mount holes

- For all keys in classic keyboard, add option for either through-hole or SMT
diodes and resistors.
Other:
- board text added: "Unified Keyboard Rev 1.8 http://osiweb.org Cherry Key Aligner"
- board text removed: "Unified Keyboard Rev 1.7 http://osiweb.org Cherry Key Aligner"
Changed lines of the file:
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@@
   (title_block
     (title "Cherry Key aligner")
-    (date 2020-06-17)
-    (rev 1.7)
+    (date 2020-06-22)
+    (rev 1.8)
     (company OSIWeb.org)
   )
@@
       (effects (font (size 1 1) (thickness 0.15)))
     )
-    (fp_text user %R (at 110.75162 -87.97036) (layer F.Fab)
-      (effects (font (size 1 1) (thickness 0.15)))
-    )
-    (fp_text user OSI (at 110.49762 -97.57156) (layer F.SilkS)
-      (effects (font (size 1 1) (thickness 0.15)))
-    )
-    (fp_text user %R (at -85.03158 5.42544) (layer F.Fab)
-      (effects (font (size 1 1) (thickness 0.15)))
-    )
-    (fp_text user OSI (at -85.28558 -4.17576) (layer F.SilkS)
-      (effects (font (size 1 1) (thickness 0.15)))
-    )
-    (fp_text user %R (at 86.31682 5.65404) (layer F.Fab)
-      (effects (font (size 1 1) (thickness 0.15)))
-    )
-    (fp_text user OSI (at 86.06282 -3.94716) (layer F.SilkS)
-      (effects (font (size 1 1) (thickness 0.15)))
-    )
-    (fp_text user OSI (at 0.59182 -97.46996) (layer F.SilkS)
-      (effects (font (size 1 1) (thickness 0.15)))
-    )
-    (fp_text user %R (at 0.84582 -87.86876) (layer F.Fab)
-      (effects (font (size 1 1) (thickness 0.15)))
-    )
-    (fp_text user OSI (at -109.56798 -97.46996) (layer F.SilkS)
-      (effects (font (size 1 1) (thickness 0.15)))
-    )
-    (fp_text user %R (at -109.31398 -87.86876) (layer F.Fab)
-      (effects (font (size 1 1) (thickness 0.15)))
-    )
-    (fp_text user OSI (at 101.48062 -96.93656) (layer F.SilkS)
-      (effects (font (size 1 1) (thickness 0.15)))
-    )
-    (fp_text user %R (at 110.75162 -87.97036) (layer F.Fab)
-      (effects (font (size 1 1) (thickness 0.15)))
-    )
     (fp_circle (center 109.22 -92.71) (end 114.046 -92.71) (layer Cmts.User) (width 0.15))
     (fp_circle (center 109.22 -92.71) (end 114.3 -92.71) (layer F.CrtYd) (width 0.05))
@@
     (fp_circle (center 109.22 -97.79) (end 114.046 -97.79) (layer Cmts.User) (width 0.15))
     (fp_circle (center 109.22 -97.79) (end 114.3 -97.79) (layer F.CrtYd) (width 0.05))
-    (pad "" np_thru_hole circle (at -85.725 0.635) (size 7.112 7.112) (drill 2.032) (layers *.Cu *.Mask))
+    (fp_text user %R (at 110.75162 -87.97036) (layer F.Fab)
+      (effects (font (size 1 1) (thickness 0.15)))
+    )
+    (fp_text user OSI (at 101.48062 -96.93656) (layer F.SilkS)
+      (effects (font (size 1 1) (thickness 0.15)))
+    )
+    (fp_text user %R (at -85.03158 5.42544) (layer F.Fab)
+      (effects (font (size 1 1) (thickness 0.15)))
+    )
+    (fp_text user OSI (at -85.28558 -4.17576) (layer F.SilkS)
+      (effects (font (size 1 1) (thickness 0.15)))
+    )
+    (fp_text user %R (at 86.31682 5.65404) (layer F.Fab)
+      (effects (font (size 1 1) (thickness 0.15)))
+    )
+    (fp_text user OSI (at 86.06282 -3.94716) (layer F.SilkS)
+      (effects (font (size 1 1) (thickness 0.15)))
+    )
+    (fp_text user OSI (at 0.59182 -97.46996) (layer F.SilkS)
+      (effects (font (size 1 1) (thickness 0.15)))
+    )
+    (fp_text user %R (at 0.84582 -87.86876) (layer F.Fab)
+      (effects (font (size 1 1) (thickness 0.15)))
+    )
+    (fp_text user OSI (at -109.56798 -97.46996) (layer F.SilkS)
+      (effects (font (size 1 1) (thickness 0.15)))
+    )
+    (fp_text user %R (at -109.31398 -87.86876) (layer F.Fab)
+      (effects (font (size 1 1) (thickness 0.15)))
+    )
+    (fp_text user OSI (at 101.48062 -96.93656) (layer F.SilkS)
+      (effects (font (size 1 1) (thickness 0.15)))
+    )
+    (fp_text user %R (at 110.75162 -87.97036) (layer F.Fab)
+      (effects (font (size 1 1) (thickness 0.15)))
+    )
+    (pad "" np_thru_hole circle (at -85.725 0.635) (size 7.112 7.112) (drill 7.112) (layers *.Cu *.Mask))
     (pad "" np_thru_hole circle (at 85.725 0.635) (size 7.112 7.112) (drill 7.112) (layers *.Cu *.Mask))
     (pad "" np_thru_hole oval (at 0 -95.25) (size 7.112 12.192) (drill oval 7.112 12.192) (layers *.Cu *.Mask))
@@
   (gr_arc (start 369.57 165.99916) (end 369.57 157.988) (angle -180) (layer Edge.Cuts) (width 0.1016))
   (gr_arc (start 369.57 89.79916) (end 369.57 82.55) (angle -180) (layer Edge.Cuts) (width 0.1016))
-  (gr_text "Unified Keyboard  Rev 1.7  http://osiweb.org\nCherry Key Aligner" (at 294.767 170.307) (layer F.SilkS)
+  (gr_text "Unified Keyboard  Rev 1.8  http://osiweb.org\nCherry Key Aligner" (at 294.767 170.307) (layer F.SilkS)
     (effects (font (size 1.524 1.524) (thickness 0.1778)) (justify left))
   )
