File: hardware/keyboard-classic/Aligner-futaba/aligner-futaba.kicad_pcb (KiCad board)
At the start: 2 copper layers, 312.4 x 118.1 mm, 74 parts, among them SW1 RT Arrow, SW10 Bracket_Open, SW11 6, SW12 Y, SW13 Return, SW14 Dash, SW15 5, SW16 T, SW17 Line Feed, SW18 Colon, SW19 4, SW2 LT Arrow, SW20 R, SW21 O, SW22 0, SW23 3, SW24 E, SW25 L, SW26 9, SW27 2, SW28 W, SW29 Period, SW3 Tilde, SW30 8, SW31 1, SW32 @ (AT), SW33 Break, SW34 Rubout, SW35 R_Shift, SW36 P, SW37 Comma, SW38 K, SW39 L_Shift, SW4 I, SW40 Semicolon, SW41 M, SW42 J, SW43 Fwd_Slash, SW44 N, SW45 H, SW46 SPACE, SW47 B, SW48 G, SW49 TAB, SW5 Repeat, SW50 Z, SW51 V, SW52 F, SW53 CTRL, SW54 A, SW55 C, SW56 D, SW57 Backslash, SW58 Q, SW59 X, SW6 Bracket_Close, SW60 S, SW61 FN, SW62 ESC, SW7 7, SW8 U, SW9 Caps Lock

Commit message: tweaks for Cherry MX stabilizer posts on Futaba aligners
- Slightly narrower posts.
- slightly smaller hole, closer to end
- added mouse bites for breakaway to avoid protruding breakaway
- Applied to Sol and Classic
Parts:
- added REF**: MountingHole_2.1mm, MountingHole:MountingHole_2.1mm, F.Cu at (254.6, 74.9)
- added REF**: MountingHole_2.1mm, MountingHole:MountingHole_2.1mm, F.Cu at (250.0, 74.9)
- added REF**: MountingHole_2.1mm, MountingHole:MountingHole_2.1mm, F.Cu at (252.3, 74.9)
- added REF**: MountingHole_2.1mm, MountingHole:MountingHole_2.1mm, F.Cu at (116.7, 74.9)
- added REF**: MountingHole_2.1mm, MountingHole:MountingHole_2.1mm, F.Cu at (119.0, 74.9)
- added REF**: MountingHole_2.1mm, MountingHole:MountingHole_2.1mm, F.Cu at (114.4, 74.9)
- moved REF** 1.00 mm to (197.2, 167.0)
Other:
- outline, holes or cut-outs redrawn

Commit message: 0.05" adjustment to position of top mounting holes to match pcb
Parts:
- removed the REF** at (364.5, 78.7)
- removed the REF** at (290.8, 78.7)
- removed the REF** at (143.5, 78.7)
- added REF**: MountingHole_3.5mm, MountingHole:MountingHole_3.5mm, F.Cu at (364.5, 77.5)
- added REF**: MountingHole_3.5mm, MountingHole:MountingHole_3.5mm, F.Cu at (290.8, 77.5)
- added REF**: MountingHole_3.5mm, MountingHole:MountingHole_3.5mm, F.Cu at (143.5, 77.5)
- moved REF** 1.27 mm to (217.2, 77.5)
- moved REF** 1.27 mm to (67.3, 77.5)

Commit message: Add BOM parameter fields to apple2 and 328P encoders and classic kbd
Other:
- board text added: "Unified Keyboard Rev 1.9 http://osiweb.org Futaba Key Aligner"
- board text removed: "Unified Keyboard Rev 1.8 http://osiweb.org Futaba Key Aligner"

Commit message: Multiple fixes for keyboard PCB
- in combined CherryMX/futaba footprints, moved cherry pads down 1 mil and
futaba pads up 2 mil, to reduce risk of shortin of LED pads with futaba pad.
Adjusted all aligners accordingly

- Fixed centroid for combined diode footprint and adjusted PCB placement on
classic and SOL keyboards accordingly.

- Moved SMT pads in combined diode footprint to top layer, so pick & place file
will be usable.

- changes to futaba stabilizer design.  Longer post adapter passes through slots
in keyboard and aligner.

- Changed futaba post thickness gauge from board outline to a slot to improve
tolerance.

- Moved spacebar stabilizer bending guide to edge of PCB, in order to make it
more useful in bending PCBs.

- Changed Apple II mounting slots on classic keyboard from horizontal to
vertical orientation, to accommodate the different spacing offets due to the use
of spacers in angled mounting threads.
Parts:
- removed the REF** at (263.7, 177.4)
- removed the REF** at (116.7, 74.9)
- removed the REF** at (119.0, 74.9)
- removed the REF** at (114.4, 74.9)
- added REF**: MountingHole_2.1mm, MountingHole:MountingHole_2.1mm, F.Cu at (167.2, 67.4)
- added REF**: MountingHole_2.1mm, MountingHole:MountingHole_2.1mm, F.Cu at (120.2, 74.9)
- added REF**: MountingHole_2.1mm, MountingHole:MountingHole_2.1mm, F.Cu at (117.9, 74.9)
- added REF**: MountingHole_2.1mm, MountingHole:MountingHole_2.1mm, F.Cu at (107.1, 72.8)
- added REF**: MountingHole_2.1mm, MountingHole:MountingHole_2.1mm, F.Cu at (115.6, 74.9)
- added REF**: MountingHole_2.1mm, MountingHole:MountingHole_2.1mm, F.Cu at (241.5, 72.8)
- moved REF** 105.8 mm to (236.1, 177.9)
Other:
- outline, holes or cut-outs redrawn
- board text added: "Unified Keyboard Rev 1.10 http://osiweb.org Futaba Key Aligner"
- board text removed: "Stabilizer bend guide"
- board text removed: "Unified Keyboard Rev 1.9 http://osiweb.org Futaba Key Aligner"

Commit message: Moved Cherry MX and futaba pads farther apart in combined footprint
- Offset cherry MX pads and aligners downward 0.004" from origin

- Offset futaba pads and aligners upward -0.004" from origin

- Update footprints in classic and sol-20 pcbs and aligners

- adjust mounting slots in Sol-20 aligners to match futaba or cherry offset
Other:
- board text added: "Unified Keyboard Rev 1.11 http://osiweb.org Futaba Key Aligner"
- board text removed: "Unified Keyboard Rev 1.10 http://osiweb.org Futaba Key Aligner"
