File: hardware/keyboard-sol-integrated/kbd-sol.kicad_pcb (KiCad board)
At the start: 2 copper layers, 396.2 x 143.1 mm, 210 parts, among them J1 Outputs, J2 SOL-20, J3 Programming, SW1 Options, SW10 TAB: 1.25x, SW11 I, SW12 2, SW13 Zero, SW14 Q, SW15 O, SW16 3, SW17 Dash, SW18 W, SW19 P, SW20 4, SW21 Caret, SW22 E, SW23 AT, SW24 5, SW25 LT Bracket, SW26 R, SW27 Return: 1.5x, SW28 6, SW29 Backslash, SW30 T, SW31 Line Feed, SW32 7, SW33 RT Bracket, SW34 Y, SW35 Load, SW36 LT Ctrl, SW37 J, SW38 Upper Case: 1.5x, SW39 M, SW4 ESC: 1.75x, SW40 Shift Lock: 1.5x, SW41 K, SW42 LT Shift: 1.5x, SW43 Comma, SW44 A, SW45 L, SW46 Z, SW47 Period, SW48 S, SW49 Semicolon, SW5 8, SW50 X, SW51 Slash, SW52 D, SW53 Colon, SW54 C, SW55 RT Shift: 2x, SW56 F, SW57 DEL, SW58 V, SW59 Mode Select: 1.75x, SW6 BREAK, SW60 G, SW61 Repeat: 1.25x, SW62 B, SW63 H, SW64 RT Ctrl, SW65 N, SW66 Local, SW67 NP Dash, SW68 NP 4, SW69 NP Zero, SW7 U, SW70 Up Arrow, SW71 NP 7, SW72 NP 1, SW73 NP period, SW74 LT Arrow, SW75 NP asterisk, SW76 NP 5, SW77 NP plus, SW78 Spacebar, SW79 NP 8, SW8 1, SW80 NP 2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

Commit message: pcb file consistency update
Parts:
- added REF**: MountingHole_3.2mm_M3, MountingHole:MountingHole_3.2mm_M3, F.Cu at (256.5, 219.5)
- moved REF** 2.68 mm to (116.0, 219.5)

Commit message: Sol-20 spacebar stabilizer fix and other cleanups
- Replaced standard MX footprint with spacebar footprint, including stabilizers
- Fixed courtyard on MX footprints in library to avoid collisions
- Added a DIP switch variant with header position closer to pin 1
- moved option DIP switch/header to align header better with edge of PCB.
Parts:
- SW1: footprint unikbd:SW_DIP_SPSTx08_Piano_CTS_Series194-8MSTN_W7.62mm_P2.54mm -> unikbd:SW_DIP_SPSTx08_oriented_backward
- SW78: footprint unikbd:Key_MX -> unikbd:Key_MX_Spacebar_5.25
- moved D90 3.18 mm to (381.5, 106.3)
- moved D91 3.18 mm to (376.4, 106.3)
- moved D92 3.18 mm to (371.3, 106.3)
- moved D93 3.18 mm to (366.3, 106.3)
- moved SW1 3.18 mm to (381.5, 87.8)
- moved D86 3.17 mm to (373.9, 101.2)
- moved D87 3.17 mm to (368.8, 101.2)
- moved D88 3.17 mm to (363.7, 101.2)
- moved D89 3.17 mm to (379.0, 101.2)
Routing:
- net /Row10: track 278.7 -> 287.6 mm
- net /Row11: track 318.9 -> 324.1 mm
- net /Row12: track 291.5 -> 296.4 mm
- net /Col4: track 668.5 -> 664.3 mm
- net /encoder/Row8: track 95.9 -> 92.1 mm
- net /Col2: track 747.5 -> 744.3 mm
- net /Col7: track 525.5 -> 522.4 mm
- net /Col6: track 528.6 -> 525.4 mm
- net /Col5: track 673.5 -> 670.3 mm
- net /Col0: track 707.6 -> 704.4 mm
- net /Col1: track 825.1 -> 824.5 mm
Other:
- board text added: "SOL-20 keyboard rev 2.1"
- board text removed: "SOL-20 keyboard rev 2.0"

Commit message: Add + symbol to bottom silk of LEDs on the keyboards
Other:
- board text added: "+"

Commit message: Added silk screen annotations for connectors.
Other:
- board text added: "+5V"
- board text added: "1"
- board text added: "2"
- board text added: "3"
- board text added: "4"
- board text added: "5"
- board text added: "6"
- board text added: "7"
- board text added: "8"
- board text added: "BREAK"
- board text added: "GND"
- board text added: "LOCAL"
- board text added: "Maps: (1,2,3): 000 - Classic 100 - Classic, ALL CAPS 010 - Apple II 011 - Apple II ALL CAPS 001 - Sol-20"
- board text added: "Options: 6 - STROBE POLARITY (OPEN=NEG, CLOSED=POS) 7 - REPEAT (OPEN=DISABLED, CLOSED=ENABLED)"
- board text added: "SOL-20"
- board text added: "~RESET"
